Commit message: Pass angular velocity as error_dot

File: rm_pioneer_description/ros2_control/guard.ros2_control.xacro (robot description, xacro)
@@ -12,8 +12,10 @@
             </hardware>
             <joint name="pitch_joint">
+                <param name="effort_actuator_coefficient">-25000</param>
                 <command_interface name="effort"/>
                 <state_interface name="position"/>
             </joint>
             <joint name="yaw_joint">
+                <param name="effort_actuator_coefficient">-25000</param>
                 <command_interface name="effort"/>
                 <state_interface name="position"/>

File: rm_pioneer_description/urdf/guard.urdf.xacro (robot description, xacro)
@@ -5,8 +5,8 @@
     <xacro:include filename="$(find rm_pioneer_description)/ros2_control/guard.ros2_control.xacro" />
     <xacro:property name="pitch_joint_limit">
-        <limit lower="0.0" upper="0.5" velocity="3.0" effort="30000"/>
+        <limit lower="0.0" upper="0.5" velocity="3.0" effort="0.8"/>
     </xacro:property>
     <xacro:property name="yaw_joint_limit">
-        <limit velocity="3.0" effort="30000"/>
+        <limit velocity="3.0" effort="0.8"/>
     </xacro:property>
     <link name="base_link" />
