Commit message: Add pitch limit

File: rm_pioneer_description/urdf/guard.urdf.xacro (robot description, xacro)
@@ -60,5 +60,5 @@
         <child link="pitch_link" />
         <axis xyz="0 1 0" />
-        <limit lower="-0.6" upper="0.5" effort="1.2" velocity="31"/>
+        <limit lower="0.0" upper="0.5" effort="0" velocity="0"/>
     </joint>
     <link name="shooter_link" />

Commit message: Update effor limit

File: rm_pioneer_description/urdf/guard.urdf.xacro (robot description, xacro)
@@ -32,4 +32,5 @@
         <child link="yaw_link" />
         <axis xyz="0 0 1" />
+        <limit velocity="0" effort="30000"/>
     </joint>
     <link name="pitch_link">
@@ -60,5 +61,5 @@
         <child link="pitch_link" />
         <axis xyz="0 1 0" />
-        <limit lower="0.0" upper="0.5" effort="0" velocity="0"/>
+        <limit lower="0.0" upper="0.5" velocity="0" effort="30000"/>
     </joint>
     <link name="shooter_link" />

Commit message: Some improvement

File: rm_pioneer_description/urdf/guard.urdf.xacro (robot description, xacro)
@@ -4,4 +4,10 @@
     <!-- Import guard ros2_control description -->
     <xacro:include filename="$(find rm_pioneer_description)/ros2_control/guard.ros2_control.xacro" />
+    <xacro:property name="pitch_joint_limit">
+        <limit lower="0.0" upper="0.5" velocity="3.0" effort="30000"/>
+    </xacro:property>
+    <xacro:property name="yaw_joint_limit">
+        <limit velocity="3.0" effort="30000"/>
+    </xacro:property>
     <link name="base_link" />
     <link name="yaw_link">
@@ -32,5 +38,5 @@
         <child link="yaw_link" />
         <axis xyz="0 0 1" />
-        <limit velocity="0" effort="30000"/>
+        <xacro:insert_block name="yaw_joint_limit" />
     </joint>
     <link name="pitch_link">
@@ -61,5 +67,5 @@
         <child link="pitch_link" />
         <axis xyz="0 1 0" />
-        <limit lower="0.0" upper="0.5" velocity="0" effort="30000"/>
+        <xacro:insert_block name="pitch_joint_limit" />
     </joint>
     <link name="shooter_link" />
@@ -99,5 +105,5 @@
     <link name="camera_optical_frame" />
     <joint name="camera_optical_joint" type="fixed">
-        <origin xyz="0 0 0" rpy="${pi/2} 0 ${pi/2}" />
+        <origin xyz="0 0 0" rpy="${-pi/2} 0 ${-pi/2}" />
         <parent link="camera_base_link" />
         <child link="camera_optical_frame" />

Commit message: Adaptation for guard

File: rm_pioneer_description/urdf/guard.urdf.xacro (robot description, xacro)
@@ -5,5 +5,5 @@
     <xacro:include filename="$(find rm_pioneer_description)/ros2_control/guard.ros2_control.xacro" />
     <xacro:property name="pitch_joint_limit">
-        <limit lower="0.0" upper="0.5" velocity="3.0" effort="0.8"/>
+        <limit lower="-0.1" upper="0.5" velocity="3.0" effort="0.8"/>
     </xacro:property>
     <xacro:property name="yaw_joint_limit">
